File: layouts/led_string/led_string.kicad_pcb (KiCad board)
At the start: 2 copper layers, 19 parts

Commit message: Try to fix fuses
Connections:
- C1 pad 1: hv -> hv-1
- C2 pad 1: hv -> hv-1
- C3 pad 1: hv -> hv-1
- C4 pad 1: hv -> hv-1
- C5 pad 1: hv -> hv-1
- C6 pad 1: hv -> hv-1
- C7 pad 1: hv -> hv-1
- C8 pad 1: hv -> hv-1
- C9 pad 1: hv -> hv-1
- LED1 pad 2: line-9 -> line-2
- LED1 pad 3: hv -> hv-1
- LED1 pad 4: line-7 -> line-5
- LED2 pad 2: line-7 -> line-5
- LED2 pad 3: hv -> hv-1
- LED2 pad 4: line -> line-7
- LED3 pad 2: line -> line-7
- LED3 pad 3: hv -> hv-1
- LED3 pad 4: line-3 -> line-9
- LED4 pad 2: line-3 -> line-9
- LED4 pad 3: hv -> hv-1
- LED4 pad 4: line-2 -> line
- LED5 pad 2: line-2 -> line
- LED5 pad 3: hv -> hv-1
- LED5 pad 4: line-6 -> line-1
- LED6 pad 2: line-6 -> line-1
- LED6 pad 3: hv -> hv-1
- LED6 pad 4: line-8 -> line-4
- LED7 pad 2: line-8 -> line-4
- LED7 pad 3: hv -> hv-1
- LED7 pad 4: line-4 -> line-3
- LED8 pad 2: line-4 -> line-3
- LED8 pad 3: hv -> hv-1
- LED8 pad 4: line-5 -> line-8
- LED9 pad 2: line-5 -> line-8
- LED9 pad 3: hv -> hv-1
- U1 pad 3: hv-1 -> hv
- U1 pad 5: line-1 -> line-6
- U1 pad 6: hv-1 -> hv
- U1 pad 7: hv -> hv-1
- U1 pad 8: line-9 -> line-2
Routing:
- net hv-1: track 0.00 -> 69.6 mm
- net hv: track 69.6 -> 0.00 mm
- net line-6: track 5.42 -> 0.00 mm
- net line-1: track 0.00 -> 5.42 mm
- net line-8: track 5.42 -> 10.5 mm
- net line-5: track 10.5 -> 5.42 mm
- net line-9: track 3.13 -> 5.42 mm, vias 1 -> 0
- net line-2: track 5.42 -> 3.13 mm, vias 0 -> 1
Changed lines of the file:
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@@
             (outputdirectory "")))
     (net 0 "")
-    (net 1 "line")
-    (net 2 "line-3")
+    (net 1 "line-7")
+    (net 2 "line-9")
     (net 3 "gnd")
-    (net 4 "line-9")
-    (net 5 "hv-1")
+    (net 4 "line-2")
+    (net 5 "hv")
     (net 6 "runtime_anon[0]-line-1")
-    (net 7 "line-5")
+    (net 7 "line-8")
     (net 8 "leds[8]-line")
-    (net 9 "line-1")
-    (net 10 "line-4")
-    (net 11 "line-8")
-    (net 12 "line-2")
-    (net 13 "line-6")
-    (net 14 "hv")
+    (net 9 "line-6")
+    (net 10 "line-3")
+    (net 11 "line-4")
+    (net 12 "line")
+    (net 13 "line-1")
+    (net 14 "hv-1")
     (net 15 "runtime_anon[0]-line")
-    (net 16 "line-7")
+    (net 16 "line-5")
     (footprint "atopile:VSON8_L2.0-W2.3-P0.50-LS3.1-BL-9e6526"
         (layer "F.Cu")
@@
             (layers "F.Cu" "F.Paste" "F.Mask")
             (remove_unused_layers no)
-            (net 5 "hv-1"))
+            (net 5 "hv"))
         (pad "4" smd rect
             (at 0.76 1.55 180)
@@
             (layers "F.Cu" "F.Paste" "F.Mask")
             (remove_unused_layers no)
-            (net 9 "line-1"))
+            (net 9 "line-6"))
         (pad "6" smd rect
             (at 0.25 -1.55 180)
@@
             (layers "F.Cu" "F.Paste" "F.Mask")
             (remove_unused_layers no)
-            (net 5 "hv-1"))
+            (net 5 "hv"))
         (pad "7" smd rect
             (at -0.25 -1.55 180)
@@
             (layers "F.Cu" "F.Paste" "F.Mask")
             (remove_unused_layers no)
-            (net 14 "hv"))
+            (net 14 "hv-1"))
         (pad "8" smd rect
             (at -0.76 -1.55 180)
@@
             (layers "F.Cu" "F.Paste" "F.Mask")
             (remove_unused_layers no)
-            (net 4 "line-9")))
+            (net 4 "line-2")))
     (footprint "atopile:C0402-b3ef17"
         (layer "B.Cu")
@@
             (layers "B.Cu" "B.Paste" "B.Mask")
             (remove_unused_layers no)
-            (net 14 "hv"))
+            (net 14 "hv-1"))
         (pad "2" smd rect
             (at 0.55 0 180)
@@
             (layers "B.Cu" "B.Paste" "B.Mask")
             (remove_unused_layers no)
-            (net 4 "line-9"))
+            (net 4 "line-2"))
         (pad "3" smd rect
             (at -1.5 0.75 0)
@@
             (layers "B.Cu" "B.Paste" "B.Mask")
             (remove_unused_layers no)
-            (net 14 "hv"))
+            (net 14 "hv-1"))
         (pad "4" smd rect
             (at -1.5 -0.75 0)
@@
             (layers "B.Cu" "B.Paste" "B.Mask")
             (remove_unused_layers no)
-            (net 16 "line-7")))
+            (net 16 "line-5")))
     (footprint "atopile:LED-SMD_4P-L3.5-W2.8-BR-1-15b4e8"
         (layer "B.Cu")
@@
             (layers "B.Cu" "B.Paste" "B.Mask")
             (remove_unused_layers no)
-            (net 16 "line-7"))
+            (net 16 "line-5"))
         (pad "3" smd rect
             (at -1.5 0.75 0)
@@
             (layers "B.Cu" "B.Paste" "B.Mask")
             (remove_unused_layers no)
-            (net 14 "hv"))
+            (net 14 "hv-1"))
         (pad "4" smd rect
             (at -1.5 -0.75 0)
@@
             (layers "B.Cu" "B.Paste" "B.Mask")
             (remove_unused_layers no)
-            (net 1 "line")))
+            (net 1 "line-7")))
     (footprint "atopile:C0402-b3ef17"
         (layer "B.Cu")
@@
             (layers "B.Cu" "B.Paste" "B.Mask")
             (remove_unused_layers no)
-            (net 14 "hv"))
+            (net 14 "hv-1"))
         (pad "2" smd rect
             (at 0.55 0 180)
@@
             (layers "B.Cu" "B.Paste" "B.Mask")
             (remove_unused_layers no)
-            (net 14 "hv"))
+            (net 14 "hv-1"))
         (pad "2" smd rect
             (at 0.55 0 180)
@@
             (layers "B.Cu" "B.Paste" "B.Mask")
             (remove_unused_layers no)
-            (net 14 "hv"))
+            (net 14 "hv-1"))
         (pad "2" smd rect
             (at 0.55 0 180)
@@
             (layers "B.Cu" "B.Paste" "B.Mask")
             (remove_unused_layers no)
-            (net 11 "line-8"))
+            (net 11 "line-4"))
         (pad "3" smd rect
             (at -1.5 0.75 0)
@@
             (layers "B.Cu" "B.Paste" "B.Mask")
             (remove_unused_layers no)
-            (net 14 "hv"))
+            (net 14 "hv-1"))
         (pad "4" smd rect
             (at -1.5 -0.75 0)
@@
             (layers "B.Cu" "B.Paste" "B.Mask")
             (remove_unused_layers no)
-            (net 10 "line-4")))
+            (net 10 "line-3")))
     (footprint "atopile:C0402-b3ef17"
         (layer "B.Cu")
@@
             (layers "B.Cu" "B.Paste" "B.Mask")
             (remove_unused_layers no)
-            (net 14 "hv"))
+            (net 14 "hv-1"))
         (pad "2" smd rect
             (at 0.55 0 180)
@@
             (layers "B.Cu" "B.Paste" "B.Mask")
             (remove_unused_layers no)
-            (net 12 "line-2"))
+            (net 12 "line"))
         (pad "3" smd rect
             (at -1.5 0.75 0)
@@
             (layers "B.Cu" "B.Paste" "B.Mask")
             (remove_unused_layers no)
-            (net 14 "hv"))
+            (net 14 "hv-1"))
         (pad "4" smd rect
             (at -1.5 -0.75 0)
@@
             (layers "B.Cu" "B.Paste" "B.Mask")
             (remove_unused_layers no)
-            (net 13 "line-6")))
+            (net 13 "line-1")))
     (footprint "atopile:C0402-b3ef17"
         (layer "B.Cu")
@@
             (layers "B.Cu" "B.Paste" "B.Mask")
             (remove_unused_layers no)
-            (net 14 "hv"))
+            (net 14 "hv-1"))
         (pad "2" smd rect
             (at 0.55 0 180)
@@
             (layers "B.Cu" "B.Paste" "B.Mask")
             (remove_unused_layers no)
-            (net 1 "line"))
+            (net 1 "line-7"))
         (pad "3" smd rect
             (at -1.5 0.75 0)
@@
             (layers "B.Cu" "B.Paste" "B.Mask")
             (remove_unused_layers no)
-            (net 14 "hv"))
+            (net 14 "hv-1"))
         (pad "4" smd rect
             (at -1.5 -0.75 0)
@@
             (layers "B.Cu" "B.Paste" "B.Mask")
             (remove_unused_layers no)
-            (net 2 "line-3")))
+            (net 2 "line-9")))
     (footprint "atopile:C0402-b3ef17"
         (layer "B.Cu")
@@
             (layers "B.Cu" "B.Paste" "B.Mask")
             (remove_unused_layers no)
-            (net 14 "hv"))
+            (net 14 "hv-1"))
         (pad "2" smd rect
             (at 0.55 0 180)
@@
             (layers "B.Cu" "B.Paste" "B.Mask")
             (remove_unused_layers no)
-            (net 14 "hv"))
+            (net 14 "hv-1"))
         (pad "2" smd rect
             (at 0.55 0 180)
@@
             (layers "B.Cu" "B.Paste" "B.Mask")
             (remove_unused_layers no)
-            (net 13 "line-6"))
+            (net 13 "line-1"))
         (pad "3" smd rect
             (at -1.5 0.75 0)
@@
             (layers "B.Cu" "B.Paste" "B.Mask")
             (remove_unused_layers no)
-            (net 14 "hv"))
+            (net 14 "hv-1"))
         (pad "4" smd rect
             (at -1.5 -0.75 0)
@@
             (layers "B.Cu" "B.Paste" "B.Mask")
             (remove_unused_layers no)
-            (net 11 "line-8")))
+            (net 11 "line-4")))
     (footprint "atopile:LED-SMD_4P-L3.5-W2.8-BR-1-15b4e8"
         (layer "B.Cu")
@@
             (layers "B.Cu" "B.Paste" "B.Mask")
             (remove_unused_layers no)
-            (net 10 "line-4"))
+            (net 10 "line-3"))
         (pad "3" smd rect
             (at -1.5 0.75 0)
@@
             (layers "B.Cu" "B.Paste" "B.Mask")
             (remove_unused_layers no)
-            (net 14 "hv"))
+            (net 14 "hv-1"))
         (pad "4" smd rect
             (at -1.5 -0.75 0)
@@
             (layers "B.Cu" "B.Paste" "B.Mask")
             (remove_unused_layers no)
-            (net 7 "line-5")))
+            (net 7 "line-8")))
     (footprint "atopile:LED-SMD_4P-L3.5-W2.8-BR-1-15b4e8"
         (layer "B.Cu")
@@
             (layers "B.Cu" "B.Paste" "B.Mask")
             (remove_unused_layers no)
-            (net 7 "line-5"))
+            (net 7 "line-8"))
         (pad "3" smd rect
             (at -1.5 0.75 0)
@@
             (layers "B.Cu" "B.Paste" "B.Mask")
             (remove_unused_layers no)
-            (net 14 "hv"))
+            (net 14 "hv-1"))
         (pad "4" smd rect
             (at -1.5 -0.75 0)
@@
             (layers "B.Cu" "B.Paste" "B.Mask")
             (remove_unused_layers no)
-            (net 14 "hv"))
+            (net 14 "hv-1"))
         (pad "2" smd rect
             (at 0.55 0 180)
@@
             (layers "B.Cu" "B.Paste" "B.Mask")
             (remove_unused_layers no)
-            (net 2 "line-3"))
+            (net 2 "line-9"))
         (pad "3" smd rect
             (at -1.5 0.75 0)
@@
             (layers "B.Cu" "B.Paste" "B.Mask")
             (remove_unused_layers no)
-            (net 14 "hv"))
+            (net 14 "hv-1"))
         (pad "4" smd rect
             (at -1.5 -0.75 0)
@@
             (layers "B.Cu" "B.Paste" "B.Mask")
             (remove_unused_layers no)
-            (net 12 "line-2")))
+            (net 12 "line")))
     (via
         (at 0 34)
