File: layouts/default/default.kicad_pcb (KiCad board)
At the start: 2 copper layers, 7 parts

Commit message: Add MCU as build target
use this ato branch to fix build:
https://github.com/atopile/atopile/pull/979
Parts:
- added C1: 100nF ±10% 50V X7R, atopile:C0603-bd72f6, F.Cu at (10.0, -5.00)
- added C2: 100nF ±10% 50V X7R, atopile:C0603-bd72f6, F.Cu at (-0.50, 12.5)
- added C3: 1µF ±10% 50V X5R, atopile:C0603-bd72f6, F.Cu at (-14.2, 22.5)
- added C3: 1µF ±10% 50V X5R, atopile:C0603-bd72f6, F.Cu at (220.0, -5.00)
- added C4: 100nF ±10% 50V X7R, atopile:C0603-bd72f6, F.Cu at (-1.00, 18.2)
- added C5: 100nF ±10% 50V X7R, atopile:C0603-bd72f6, F.Cu at (-3.50, 18.8)
- added C6: 100nF ±10% 50V X7R, atopile:C0603-bd72f6, F.Cu at (-0.75, 7.75)
- added C7: 100nF ±5% 16V X7R, atopile:C0402-b3ef17, F.Cu at (270.0, -5.00)
- added H1: , MountingHole:MountingHole_2.2mm_M2_Pad, F.Cu at (-6.50, 2.50)
- added H2: , MountingHole:MountingHole_2.2mm_M2_Pad, F.Cu at (7.50, 69.5)
- added H3: , MountingHole:MountingHole_2.2mm_M2_Pad, F.Cu at (-7.50, 69.5)
- added J1: , atopile:USB-C-TH_TYPE-C-USB-14P-1a34cb, F.Cu at (-0.25, 72.5)
- added J2: , atopile:CONN-SMD_ZH1.5-4AB-9aedad, F.Cu at (26.5, 8.00)
- added LED1: , atopile:LED-SMD_4P-L3.5-W2.8-BR-1-15b4e8, F.Cu at (-48.0, 39.0)
- added LED2: , atopile:LED-SMD_4P-L3.5-W2.8-BR-1-15b4e8, F.Cu at (-48.0, 42.5)
- added LED3: , atopile:LED-SMD_4P-L3.5-W2.8-BR-1-15b4e8, F.Cu at (-48.0, 46.0)
- added LED4: , atopile:LED-SMD_4P-L3.5-W2.8-BR-1-15b4e8, F.Cu at (-48.0, 49.5)
- added LED5: , atopile:LED-SMD_4P-L3.5-W2.8-BR-1-15b4e8, F.Cu at (-48.0, 53.0)
- added R10: 5.1kΩ ±1% 100mW, atopile:R0603-ebcab9, F.Cu at (130.0, -5.00)
- added R11: 1MΩ ±1% 250mW, atopile:R1206-bdb864, F.Cu at (190.0, -5.00)
- added R12: 10kΩ ±1% 100mW, atopile:R0603-ebcab9, F.Cu at (9.75, 16.0)
- added R13: 10kΩ ±1% 100mW, atopile:R0603-ebcab9, F.Cu at (13.5, 12.8)
- added R4: 10kΩ ±1% 100mW, atopile:R0603-ebcab9, F.Cu at (-9.40, 22.6)
- added R5: 10kΩ ±1% 100mW, atopile:R0603-ebcab9, F.Cu at (-14.0, 17.0)
- added R6: 10kΩ ±1% 100mW, atopile:R0603-ebcab9, F.Cu at (-11.8, 22.5)
- added R7: 10kΩ ±1% 100mW, atopile:R0603-ebcab9, F.Cu at (-3.50, 10.8)
- added R8: 10kΩ ±1% 100mW, atopile:R0603-ebcab9, F.Cu at (1.00, 7.75)
- added R9: 5.1kΩ ±1% 100mW, atopile:R0603-ebcab9, F.Cu at (80.0, -5.00)
- added U1: , atopile:LGA-20_L10.1-W10.1-P1.25-TL-a13bdd, F.Cu at (11.8, 0.75)
- added U2: LDO Vin max Iq, atopile:SOT-23-5_L3.0-W1.7-P0.95-LS2.8-BL-01dfeb, F.Cu at (410.0, -5.00)
- added U3: LDO Vin max Iq, atopile:SOT-23-5_L3.0-W1.7-P0.95-LS2.8-BL-01dfeb, F.Cu at (160.0, -5.00)
- added U4: , atopile:WSOF-6_L2.6-W1.6-P0.50-TL-EP-b2dfd8, B.Cu at (0.00, 8.50)
- added U5: , atopile:WIFIM-SMD_ESP32-C3-MINI-MINI-1U-1cb675, F.Cu at (-11.0, 14.0)
- added U6: , atopile:VSON8_L2.0-W2.3-P0.50-LS3.1-BL-9e6526, F.Cu at (26.5, 14.0)
- added U7: , atopile:SENSORM-TH_HLK-LD2410B-P-2a325e, F.Cu at (310.0, -5.00)
- added U8: , atopile:VSON8_L2.0-W2.3-P0.50-LS3.1-BL-9e6526, F.Cu at (162.0, 34.0)
- added X1: , atopile:CONN-SMD_4P-P1.00_SM04B-SRSS-TB-LF-SN-d36980, F.Cu at (252.5, 61.0)
- R1: value 5.1kΩ ±1% 62.5mW -> 10kΩ ±1% 100mW; footprint atopile:R0402-56259e -> atopile:R0603-ebcab9
- moved R1 190.0 mm to (200.0, -5.00)
- moved R3 47.3 mm to (-0.50, 14.2)
- moved D1 35.1 mm to (13.5, 14.5)
- moved D2 35.1 mm to (16.8, 14.8)
- moved FanConnector1 35.1 mm to (13.5, 18.0)
- moved Q1 35.1 mm to (9.50, 13.5)
- moved R2 4.25 mm to (40.0, -5.00), turned to 0 degrees
Connections:
- net fan_connector-gnd-2 renamed vindriktning_interface.fan_controller-gnd
- net fan_connector.fan_connector.footprint.pins[2].net-net renamed vindriktning_interface.fan_controller.fan_connector.footprint.pins[2].net-net
- net fan_connector.fan_connector.footprint.pins[3].net-net renamed vindriktning_interface.fan_controller.fan_connector.footprint.pins[3].net-net
- D1 pad 1: hv -> vindriktning_interface.fan_controller-hv
- D1 pad 2: fan_connector-gnd-1 -> vindriktning_interface.fan_controller-gnd-1
- D2 pad 1: hv -> vindriktning_interface.fan_controller-hv
- FanConnector1 pad 1: fan_connector-gnd-1 -> vindriktning_interface.fan_controller-gnd-1
- FanConnector1 pad 2: hv -> vindriktning_interface.fan_controller-hv
- Q1 pad 1: line -> line-5
- Q1 pad 2: fan_connector-gnd-1 -> vindriktning_interface.fan_controller-gnd-1
- R1 pad 1: r-net-1 -> line-9
- R1 pad 2: r-net -> hv
- R2 pad 2: fan_connector-gnd -> hv
- R3 pad 1: cathode -> mcu.mcu.boot_switch-line
- R3 pad 2: fan_connector-gnd-1 -> mcu.mcu.boot_switch.lp_filter-line
Routing:
- net vindriktning_interface.fan_controller-gnd-1: track 0.00 -> 6.53 mm
- net fan_connector-gnd-1: track 6.53 -> 0.00 mm
- net vindriktning_interface.fan_controller-hv: track 0.00 -> 5.20 mm
- net hv: track 5.20 -> 0.00 mm
- net line-5: track 0.00 -> 1.55 mm
- net line: track 1.55 -> 0.00 mm

Commit message: Migrate layout partially
omit routing and zones amongst others
Parts:
- removed the C3 at (220.0, -5.00)
- moved U7 130.0 mm to (180.0, -5.00)
- moved R5 22.8 mm to (-3.00, -3.00), turned to 0 degrees
Connections:
- C1 pad 1: hv -> hv-2
- C3 pad 1: hv-3 -> hv-1
- D1 pad 2: vindriktning_interface.fan_controller-gnd-1 -> vindriktning_interface.fan_controller-gnd
- FanConnector1 pad 1: vindriktning_interface.fan_controller-gnd-1 -> vindriktning_interface.fan_controller-gnd
- J1 pad 10: line-6 -> line-3
- J1 pad 11: line-10 -> line-9
- J1 pad 3: line-6 -> line-3
- J1 pad 4: line-10 -> line-9
- J2 pad 3: hv-2 -> hv-3
- LED1 pad 2: led_string-line -> led_string-line-2
- LED1 pad 3: hv-2 -> hv-3
- LED2 pad 3: hv-2 -> hv-3
- LED3 pad 3: hv-2 -> hv-3
- LED3 pad 4: led_string-line-2 -> led_string-line
- LED4 pad 2: led_string-line-2 -> led_string-line
- LED4 pad 3: hv-2 -> hv-3
- LED5 pad 3: hv-2 -> hv-3
- Q1 pad 1: line-5 -> line-4
- Q1 pad 2: vindriktning_interface.fan_controller-gnd-1 -> vindriktning_interface.fan_controller-gnd
- Q1 pad 3: vindriktning_interface.fan_controller-gnd -> vindriktning_interface.fan_controller-gnd-1
- R1 pad 1: line-9 -> line-10
- R1 pad 2: hv -> hv-2
- R12 pad 1: line-5 -> line-4
- R13 pad 2: vindriktning_interface.fan_controller-gnd-1 -> vindriktning_interface.fan_controller-gnd
- R2 pad 1: line -> line-7
- R2 pad 2: hv -> hv-2
- R4 pad 1: mcu.mcu-line -> mcu.mcu-line-1
- R4 pad 2: hv-3 -> hv-1
- R5 pad 2: mcu.mcu-line-1 -> mcu.mcu-line
- R6 pad 1: line-9 -> line-10
- R6 pad 2: hv-3 -> hv-1
- R7 pad 1: line-1 -> line-6
- R7 pad 2: hv-3 -> hv-1
- U1 pad 10: line -> line-7
- U1 pad 19: hv -> hv-2
- U1 pad 7: hv -> hv-2
- U1 pad 9: line-9 -> line-10
- U2 pad 1: hv-2 -> hv-3
- U2 pad 3: hv-2 -> hv-3
- U2 pad 5: hv-3 -> hv-1
- U3 pad 1: hv-2 -> hv-3
- U3 pad 3: hv-2 -> hv-3
- U3 pad 5: hv -> hv-2
- U4 pad 1: hv -> hv-2
- U4 pad 2: lux_sensor.ic-line -> lux_sensor.ic-line-1
- U4 pad 4: line -> line-7
- U4 pad 5: lux_sensor.ic-line-2 -> lux_sensor.ic-line
- U4 pad 6: line-9 -> line-10
- U4 pad 7: lux_sensor.ic-line-1 -> lux_sensor.ic-line-2
- U5 pad 13: mcu.mcu-line-1 -> mcu.mcu-line
- U5 pad 16: mcu.mcu.esp32_c3_mini_1.ic-line -> mcu.mcu.esp32_c3_mini_1.ic-line-1
- U5 pad 18: line-5 -> line-4
- U5 pad 19: line-2 -> line-8
- U5 pad 20: line-8 -> line
- U5 pad 21: mcu.mcu.esp32_c3_mini_1.ic-line-1 -> mcu.mcu.esp32_c3_mini_1.ic-line
- U5 pad 22: line-1 -> line-6
- U5 pad 23: line-3 -> line-2
- U5 pad 26: line-6 -> line-3
- U5 pad 27: line-10 -> line-9
- U5 pad 3: hv-3 -> hv-1
- U5 pad 30: line-4 -> line-1
- U5 pad 31: line-7 -> line-5
- U5 pad 5: line-9 -> line-10
- U5 pad 6: line -> line-7
- U5 pad 8: mcu.mcu-line -> mcu.mcu-line-1
- U6 pad 3: hv -> hv-2
- U6 pad 4: line-3 -> line-2
- U6 pad 5: line-1 -> line-6
- U6 pad 6: hv -> hv-2
- U6 pad 7: hv-2 -> hv-3
- U7 pad 1: line-8 -> line
- U7 pad 2: line-7 -> line-5
- U7 pad 3: line-4 -> line-1
- U7 pad 5: hv-2 -> hv-3
- U8 pad 3: hv -> hv-2
- U8 pad 5: line-2 -> line-8
- U8 pad 6: hv -> hv-2
- U8 pad 7: hv-2 -> hv-3
- U8 pad 8: led_string-line -> led_string-line-2
- X1 pad 2: hv-1 -> hv
- X1 pad 3: line -> line-7
- X1 pad 4: line-9 -> line-10
Routing:
- net vindriktning_interface.fan_controller-gnd-1: track 6.53 -> 0.00 mm
- net vindriktning_interface.fan_controller-gnd: track 0.00 -> 6.53 mm
- net line-5: track 1.55 -> 0.00 mm
- net line-4: track 0.00 -> 1.55 mm
Other:
- board outline added: 38 x 75 mm
- board text added: "Vindriktning"
- board text added: "a4eeddd"

Commit message: Regenerate layouts
Parts:
- moved U1 49.5 mm to (-35.6, 14.8)
- moved U6 15.0 mm to (11.5, 13.0), turned to 90 degrees
- moved LED1 14.1 mm to (-34.0, 41.0)
- moved LED2 14.1 mm to (-34.0, 44.5)
- moved LED3 14.1 mm to (-34.0, 48.0)
- moved LED4 14.1 mm to (-34.0, 51.5)
- moved LED5 14.1 mm to (-34.0, 55.0)
- moved U8 14.1 mm to (176.0, 36.0)
- moved J2 14.0 mm to (12.5, 8.40)
- moved D1 3.64 mm to (12.5, 18.0)
- moved D2 3.64 mm to (15.8, 18.2)
- moved FanConnector1 3.64 mm to (12.5, 21.5)
- moved Q1 3.64 mm to (8.50, 17.0)
- moved R12 3.64 mm to (8.75, 19.5)
- moved R13 3.64 mm to (12.5, 16.2)
Connections:
- net mcu.mcu.low_speed_crystal_clock-net renamed unnamed[0]
- C1 pad 1: hv-2 -> hv-1
- C3 pad 1: hv-1 -> hv-3
- C5 pad 1: mcu.mcu-line-2 -> mcu.mcu-line
- D1 pad 2: vindriktning_interface.fan_controller-gnd -> vindriktning_interface.fan_controller-gnd-1
- FanConnector1 pad 1: vindriktning_interface.fan_controller-gnd -> vindriktning_interface.fan_controller-gnd-1
- J1 pad 10: line-3 -> line-1
- J1 pad 11: line-9 -> line-7
- J1 pad 3: line-3 -> line-1
- J1 pad 4: line-9 -> line-7
- J2 pad 3: hv-3 -> hv
- LED1 pad 2: led_string-line-2 -> led_string-line-4
- LED1 pad 3: hv-3 -> hv
- LED1 pad 4: led_string-line-4 -> led_string-line-3
- LED2 pad 2: led_string-line-4 -> led_string-line-3
- LED2 pad 3: hv-3 -> hv
- LED2 pad 4: led_string-line-1 -> led_string-line-2
- LED3 pad 2: led_string-line-1 -> led_string-line-2
- LED3 pad 3: hv-3 -> hv
- LED4 pad 3: hv-3 -> hv
- LED4 pad 4: led_string-line-3 -> led_string-line-1
- LED5 pad 2: led_string-line-3 -> led_string-line-1
- LED5 pad 3: hv-3 -> hv
- Q1 pad 1: line-4 -> line-10
- Q1 pad 2: vindriktning_interface.fan_controller-gnd -> vindriktning_interface.fan_controller-gnd-1
- Q1 pad 3: vindriktning_interface.fan_controller-gnd-1 -> vindriktning_interface.fan_controller-gnd
- R1 pad 1: line-10 -> line-9
- R1 pad 2: hv-2 -> hv-1
- R12 pad 1: line-4 -> line-10
- R13 pad 2: vindriktning_interface.fan_controller-gnd -> vindriktning_interface.fan_controller-gnd-1
- R2 pad 1: line-7 -> line-3
- R2 pad 2: hv-2 -> hv-1
- R4 pad 2: hv-1 -> hv-3
- R5 pad 2: mcu.mcu-line -> mcu.mcu-line-2
- R6 pad 1: line-10 -> line-9
- R6 pad 2: hv-1 -> hv-3
- R7 pad 1: line-6 -> line-4
- R7 pad 2: hv-1 -> hv-3
- U1 pad 10: line-7 -> line-3
- U1 pad 19: hv-2 -> hv-1
- U1 pad 7: hv-2 -> hv-1
- U1 pad 9: line-10 -> line-9
- U2 pad 1: hv-3 -> hv
- U2 pad 3: hv-3 -> hv
- U2 pad 5: hv-1 -> hv-3
- U3 pad 1: hv-3 -> hv
- U3 pad 3: hv-3 -> hv
- U3 pad 5: hv-2 -> hv-1
- U4 pad 1: hv-2 -> hv-1
- U4 pad 2: lux_sensor.ic-line-1 -> lux_sensor.ic-line-2
- U4 pad 4: line-7 -> line-3
- U4 pad 5: lux_sensor.ic-line -> lux_sensor.ic-line-1
- U4 pad 6: line-10 -> line-9
- U4 pad 7: lux_sensor.ic-line-2 -> lux_sensor.ic-line
- U5 pad 12: mcu.mcu-line-2 -> mcu.mcu-line
- U5 pad 13: mcu.mcu-line -> mcu.mcu-line-2
- U5 pad 18: line-4 -> line-10
- U5 pad 20: line -> line-2
- U5 pad 22: line-6 -> line-4
- U5 pad 23: line-2 -> line-5
- U5 pad 26: line-3 -> line-1
- U5 pad 27: line-9 -> line-7
- U5 pad 3: hv-1 -> hv-3
- U5 pad 30: line-1 -> line
- U5 pad 31: line-5 -> line-6
- U5 pad 5: line-10 -> line-9
- U5 pad 6: line-7 -> line-3
- U6 pad 3: hv-2 -> hv-1
- U6 pad 4: line-2 -> line-5
- U6 pad 5: line-6 -> line-4
- U6 pad 6: hv-2 -> hv-1
- U6 pad 7: hv-3 -> hv
- U7 pad 1: line -> line-2
- U7 pad 2: line-5 -> line-6
- U7 pad 3: line-1 -> line
- U7 pad 5: hv-3 -> hv
- U8 pad 1: led_string.runtime_anon[0]-line -> led_string.runtime_anon[0]-line-1
- U8 pad 3: hv-2 -> hv-1
- U8 pad 4: led_string.runtime_anon[0]-line-1 -> led_string.runtime_anon[0]-line
- U8 pad 6: hv-2 -> hv-1
- U8 pad 7: hv-3 -> hv
- U8 pad 8: led_string-line-2 -> led_string-line-4
- X1 pad 2: hv -> hv-2
- X1 pad 3: line-7 -> line-3
- X1 pad 4: line-10 -> line-9
Routing:
- net vindriktning_interface.fan_controller-gnd: track 6.53 -> 0.00 mm
- net vindriktning_interface.fan_controller-gnd-1: track 0.00 -> 6.53 mm
- net line-4: track 1.55 -> 0.00 mm
- net line-10: track 0.00 -> 1.55 mm
Other:
- board text added: "d9546bd"

Commit message: Update layouts
Parts:
- D2: value infV -> (none)
- moved U8 173.8 mm to (4.70, 6.50)
- moved LED1 48.4 mm to (0.00, 6.50)
- moved LED2 45.8 mm to (0.00, 13.8)
- moved LED3 43.4 mm to (0.00, 21.0)
- moved LED4 41.2 mm to (0.00, 28.2)
- moved LED5 39.2 mm to (0.00, 35.5)
- moved U1 8.54 mm to (-39.4, 7.15)
Connections:
- net unnamed[0] renamed mcu.mcu.low_speed_crystal_clock-net
- C1 pad 1: hv-1 -> hv
- C1 pad 2: gnd -> gnd-1
- C3 pad 2: gnd -> gnd-1
- C4 pad 2: gnd -> gnd-1
- C5 pad 1: mcu.mcu-line -> mcu.mcu-line-1
- C5 pad 2: gnd -> gnd-1
- C7 pad 2: gnd -> gnd-1
- J1 pad 1: gnd -> gnd-1
- J1 pad 10: line-1 -> line-9
- J1 pad 11: line-7 -> line-6
- J1 pad 14: gnd -> gnd-1
- J1 pad 3: line-1 -> line-9
- J1 pad 4: line-7 -> line-6
- J1 pad 7: gnd -> gnd-1
- J1 pad 8: gnd -> gnd-1
- J2 pad 1: vindriktning_interface-line -> vindriktning_interface-line-1
- J2 pad 2: vindriktning_interface-line-1 -> vindriktning_interface-line
- J2 pad 3: hv -> hv-1
- J2 pad 4: gnd -> gnd-1
- LED1 pad 1: gnd -> gnd-1
- LED1 pad 2: led_string-line-4 -> led_string-line-1
- LED1 pad 3: hv -> hv-1
- LED1 pad 4: led_string-line-3 -> led_string-line
- LED2 pad 1: gnd -> gnd-1
- LED2 pad 2: led_string-line-3 -> led_string-line
- LED2 pad 3: hv -> hv-1
- LED2 pad 4: led_string-line-2 -> led_string-line-3
- LED3 pad 1: gnd -> gnd-1
- LED3 pad 2: led_string-line-2 -> led_string-line-3
- LED3 pad 3: hv -> hv-1
- LED3 pad 4: led_string-line -> led_string-line-4
- LED4 pad 1: gnd -> gnd-1
- LED4 pad 2: led_string-line -> led_string-line-4
- LED4 pad 3: hv -> hv-1
- LED4 pad 4: led_string-line-1 -> led_string-line-2
- LED5 pad 1: gnd -> gnd-1
- LED5 pad 2: led_string-line-1 -> led_string-line-2
- LED5 pad 3: hv -> hv-1
- Q1 pad 1: line-10 -> line
- R1 pad 1: line-9 -> line-3
- R1 pad 2: hv-1 -> hv
- R10 pad 2: gnd -> gnd-1
- R11 pad 2: gnd -> gnd-1
- R12 pad 1: line-10 -> line
- R12 pad 2: gnd -> gnd-1
- R2 pad 1: line-3 -> line-4
- R2 pad 2: hv-1 -> hv
- R4 pad 1: mcu.mcu-line-1 -> mcu.mcu-line
- R6 pad 1: line-9 -> line-3
- R7 pad 1: line-4 -> line-2
- R9 pad 2: gnd -> gnd-1
- U1 pad 10: line-3 -> line-4
- U1 pad 19: hv-1 -> hv
- U1 pad 20: gnd -> gnd-1
- U1 pad 21: gnd -> gnd-1
- U1 pad 6: gnd -> gnd-1
- U1 pad 7: hv-1 -> hv
- U1 pad 9: line-9 -> line-3
- U2 pad 1: hv -> hv-1
- U2 pad 2: gnd -> gnd-1
- U2 pad 3: hv -> hv-1
- U3 pad 1: hv -> hv-1
- U3 pad 2: gnd -> gnd-1
- U3 pad 3: hv -> hv-1
- U3 pad 5: hv-1 -> hv
- U4 pad 1: hv-1 -> hv
- U4 pad 2: lux_sensor.ic-line-2 -> lux_sensor.ic-line-1
- U4 pad 3: gnd -> gnd-1
- U4 pad 4: line-3 -> line-4
- U4 pad 5: lux_sensor.ic-line-1 -> lux_sensor.ic-line
- U4 pad 6: line-9 -> line-3
- U4 pad 7: lux_sensor.ic-line -> lux_sensor.ic-line-2
- U5 pad 1: gnd -> gnd-1
- U5 pad 11: gnd -> gnd-1
- U5 pad 12: mcu.mcu-line -> mcu.mcu-line-1
- U5 pad 14: gnd -> gnd-1
- U5 pad 18: line-10 -> line
- U5 pad 19: line-8 -> line-7
- U5 pad 2: gnd -> gnd-1
- U5 pad 20: line-2 -> line-8
- U5 pad 22: line-4 -> line-2
- U5 pad 23: line-5 -> line-1
- U5 pad 26: line-1 -> line-9
- U5 pad 27: line-7 -> line-6
- U5 pad 30: line -> line-5
- U5 pad 31: line-6 -> line-10
- U5 pad 36: gnd -> gnd-1
- U5 pad 37: gnd -> gnd-1
- U5 pad 38: gnd -> gnd-1
- U5 pad 39: gnd -> gnd-1
- U5 pad 40: gnd -> gnd-1
- U5 pad 41: gnd -> gnd-1
- U5 pad 42: gnd -> gnd-1
- U5 pad 43: gnd -> gnd-1
- U5 pad 44: gnd -> gnd-1
- U5 pad 45: gnd -> gnd-1
- U5 pad 46: gnd -> gnd-1
- U5 pad 47: gnd -> gnd-1
- U5 pad 48: gnd -> gnd-1
- U5 pad 49: gnd -> gnd-1
- U5 pad 5: line-9 -> line-3
- U5 pad 50: gnd -> gnd-1
- U5 pad 51: gnd -> gnd-1
- U5 pad 52: gnd -> gnd-1
- U5 pad 53: gnd -> gnd-1
- U5 pad 54: gnd -> gnd-1
- U5 pad 55: gnd -> gnd-1
- U5 pad 56: gnd -> gnd-1
- U5 pad 57: gnd -> gnd-1
- U5 pad 58: gnd -> gnd-1
- U5 pad 59: gnd -> gnd-1
- U5 pad 6: line-3 -> line-4
- U5 pad 60: gnd -> gnd-1
- U5 pad 61: gnd -> gnd-1
- U5 pad 8: mcu.mcu-line-1 -> mcu.mcu-line
- U6 pad 1: vindriktning_interface-line-1 -> vindriktning_interface-line
- U6 pad 2: gnd -> gnd-1
- U6 pad 3: hv-1 -> hv
- U6 pad 4: line-5 -> line-1
- U6 pad 5: line-4 -> line-2
- U6 pad 6: hv-1 -> hv
- U6 pad 7: hv -> hv-1
- U6 pad 8: vindriktning_interface-line -> vindriktning_interface-line-1
- U7 pad 1: line-2 -> line-8
- U7 pad 2: line-6 -> line-10
- U7 pad 3: line -> line-5
- U7 pad 4: gnd -> gnd-1
- U7 pad 5: hv -> hv-1
- U8 pad 2: gnd -> gnd-1
- U8 pad 3: hv-1 -> hv
- U8 pad 5: line-8 -> line-7
- U8 pad 6: hv-1 -> hv
- U8 pad 7: hv -> hv-1
- U8 pad 8: led_string-line-4 -> led_string-line-1
- X1 pad 1: gnd-1 -> gnd
- X1 pad 3: line-3 -> line-4
- X1 pad 4: line-9 -> line-3
Routing:
- net led_string-line-4: track 0.00 -> 6.99 mm
- net led_string-line-3: track 0.00 -> 6.99 mm
- net led_string-line-2: track 0.00 -> 6.99 mm
- net led_string-line: track 0.00 -> 6.99 mm
- net led_string-line-1: track 0.00 -> 2.77 mm
- net line-10: track 1.55 -> 0.00 mm
- net line: track 0.00 -> 1.55 mm
Other:
- board text added: "069b639"
- board text added: "380a7ca"
